Commit message: new drone orientation in onshape with forward aligned with x-axis and centre of drone on origin

File: cad_src/drone.urdf (robot description, URDF)
Before this commit: robot drone, 11 links, 10 joints
Joints:
- joint joint_camera: origin xyz=-0.000969365 -0.0193568 -0.00117609 rpy=-1.5708 -0 -0 -> xyz=0.0197234 -8.03059e-05 0.01 rpy=-1.5708 -0 1.5708
- joint joint_imu: origin xyz=-0.000969365 0.000643159 -0.00617609 rpy=3.14159 -0 0 -> xyz=-0.000276567 -8.03059e-05 0.005 rpy=3.14159 -0 1.5708
- joint joint_motor_FL: origin xyz=0.0890306 -0.0893568 -0.0111761 rpy=3.14159 -0 0 -> xyz=0.0897234 0.0899197 0 rpy=3.14159 -0 1.5708
- joint joint_motor_FR: origin xyz=-0.0909694 -0.0893568 -0.0111761 rpy=3.14159 -0 0 -> xyz=0.0897234 -0.0900803 0 rpy=3.14159 -0 1.5708
- joint joint_motor_RL: origin xyz=0.0890306 0.0906432 -0.0111761 rpy=3.14159 -0 0 -> xyz=-0.0902766 0.0899197 0 rpy=3.14159 -0 1.5708
- joint joint_motor_RR: origin xyz=-0.0909694 0.0906432 -0.0111761 rpy=3.14159 -0 0 -> xyz=-0.0902766 -0.0900803 0 rpy=3.14159 -0 1.5708
- joint joint_rotor_FL: origin xyz=0 0 -0.02 rpy=3.14159 -0 0 -> xyz=0 0 -0.02 rpy=3.14159 -0 1.5708
- joint joint_rotor_FR: origin xyz=0 0 -0.02 rpy=3.14159 -0 0 -> xyz=0 0 -0.02 rpy=3.14159 -0 1.5708
- joint joint_rotor_RL: origin xyz=0 -0 -0.02 rpy=3.14159 -0 -0.160013 -> xyz=0 -0 -0.02 rpy=3.14159 -0 1.41078
- joint joint_rotor_RR: origin xyz=0 0 -0.02 rpy=3.14159 -0 0 -> xyz=-0 0 -0.02 rpy=3.14159 -0 1.5708
