Commit message: numerous changes to structure, add CMakeLists file for build, add package.xml file for identification, modified scripsts to use relative paths rather than absolute.

File: urdf/drone.urdf.xacro (robot description, xacro)
@@ -25,8 +25,8 @@
     <xacro:property name="l_motor_rl_vis_coll_orig_rpy" value="3.14159 -0 0" />
     <xacro:property name="l_motor_rr_vis_coll_orig_rpy" value="3.14159 -0 0" />
-    <xacro:property name="l_motor_fl_mesh" value="package://assets/link_motor_fl.stl" />
-    <xacro:property name="l_motor_fr_mesh" value="package://assets/link_motor_fr.stl" />
-    <xacro:property name="l_motor_rl_mesh" value="package://assets/link_motor_rl.stl" />
-    <xacro:property name="l_motor_rr_mesh" value="package://assets/link_motor_rr.stl" />
+    <xacro:property name="l_motor_fl_mesh" value="package://meshes/link_motor_fl.stl" />
+    <xacro:property name="l_motor_fr_mesh" value="package://meshes/link_motor_fr.stl" />
+    <xacro:property name="l_motor_rl_mesh" value="package://meshes/link_motor_rl.stl" />
+    <xacro:property name="l_motor_rr_mesh" value="package://meshes/link_motor_rr.stl" />
     <xacro:property name="j_motor_fr_orig_xyz" value="-0.0909694 -0.0893568 -0.0111761" />
     <xacro:property name="j_motor_fr_orig_rpy" value="3.14159 -0 0" />
@@ -69,8 +69,8 @@
     <xacro:property name="l_rotor_rl_vis_coll_orig_rpy" value="0 -0 0" />
     <xacro:property name="l_rotor_rr_vis_coll_orig_rpy" value="0 -0 0" />
-    <xacro:property name="l_rotor_fl_mesh" value="package://assets/link_rotor_fl.stl" />
-    <xacro:property name="l_rotor_fr_mesh" value="package://assets/link_rotor_fr.stl" />
-    <xacro:property name="l_rotor_rl_mesh" value="package://assets/link_rotor_rl.stl" />
-    <xacro:property name="l_rotor_rr_mesh" value="package://assets/link_rotor_rr.stl" />
+    <xacro:property name="l_rotor_fl_mesh" value="package://meshes/link_rotor_fl.stl" />
+    <xacro:property name="l_rotor_fr_mesh" value="package://meshes/link_rotor_fr.stl" />
+    <xacro:property name="l_rotor_rl_mesh" value="package://meshes/link_rotor_rl.stl" />
+    <xacro:property name="l_rotor_rr_mesh" value="package://meshes/link_rotor_rr.stl" />
     <xacro:property name="j_rotor_fr_orig_xyz" value="0 0 -0.02" />
     <xacro:property name="j_rotor_fr_orig_rpy" value="3.14159 -0 0" />
@@ -181,5 +181,5 @@
       <origin xyz="-0.000969365 0.000643159 -0.0111761" rpy="0 -0 0" />
       <geometry>
-        <mesh filename="package://assets/link_drone_body.stl" />
+        <mesh filename="package://meshes/link_drone_body.stl" />
       </geometry>
       <material name="link_drone_body_material">
@@ -190,5 +190,5 @@
       <origin xyz="-0.000969365 0.000643159 -0.0111761" rpy="0 -0 0" />
       <geometry>
-        <mesh filename="package://assets/link_drone_body.stl" />
+        <mesh filename="package://meshes/link_drone_body.stl" />
       </geometry>
     </collision>
@@ -203,5 +203,5 @@
       <origin xyz="-0 -0 0" rpy="3.14159 -0 0" />
       <geometry>
-        <mesh filename="package://assets/link_imu.stl" />
+        <mesh filename="package://meshes/link_imu.stl" />
       </geometry>
       <material name="link_imu_material">
@@ -212,5 +212,5 @@
       <origin xyz="-0 -0 0" rpy="3.14159 -0 0" />
       <geometry>
-        <mesh filename="package://assets/link_imu.stl" />
+        <mesh filename="package://meshes/link_imu.stl" />
       </geometry>
     </collision>
@@ -225,5 +225,5 @@
       <origin xyz="-0 -0 -0" rpy="1.5708 -0 0" />
       <geometry>
-        <mesh filename="package://assets/link_camera.stl" />
+        <mesh filename="package://meshes/link_camera.stl" />
       </geometry>
       <material name="link_camera_material">
@@ -234,5 +234,5 @@
       <origin xyz="-0 -0 -0" rpy="1.5708 -0 0" />
       <geometry>
-        <mesh filename="package://assets/link_camera.stl" />
+        <mesh filename="package://meshes/link_camera.stl" />
       </geometry>
     </collision>
