Commit message: fixing path error in drone.urdf.xacro

File: urdf/drone.urdf.xacro (robot description, xacro)
@@ -25,8 +25,8 @@
   <xacro:property name="l_motor_rl_vis_coll_orig_rpy" value="3.14159 -0 0" />
   <xacro:property name="l_motor_rr_vis_coll_orig_rpy" value="3.14159 -0 0" />
-  <xacro:property name="l_motor_fl_mesh" value="package://meshes/link_motor_fl.stl" />
-  <xacro:property name="l_motor_fr_mesh" value="package://meshes/link_motor_fr.stl" />
-  <xacro:property name="l_motor_rl_mesh" value="package://meshes/link_motor_rl.stl" />
-  <xacro:property name="l_motor_rr_mesh" value="package://meshes/link_motor_rr.stl" />
+  <xacro:property name="l_motor_fl_mesh" value="package://enph353-comp-drone/meshes/link_motor_fl.stl" />
+  <xacro:property name="l_motor_fr_mesh" value="package://enph353-comp-drone/meshes/link_motor_fr.stl" />
+  <xacro:property name="l_motor_rl_mesh" value="package://enph353-comp-drone/meshes/link_motor_rl.stl" />
+  <xacro:property name="l_motor_rr_mesh" value="package://enph353-comp-drone/meshes/link_motor_rr.stl" />
   <xacro:property name="j_motor_fr_orig_xyz" value="-0.0909694 -0.0893568 -0.0111761" />
   <xacro:property name="j_motor_fr_orig_rpy" value="3.14159 -0 0" />
@@ -69,8 +69,8 @@
   <xacro:property name="l_rotor_rl_vis_coll_orig_rpy" value="0 -0 0" />
   <xacro:property name="l_rotor_rr_vis_coll_orig_rpy" value="0 -0 0" />
-  <xacro:property name="l_rotor_fl_mesh" value="package://meshes/link_rotor_fl.stl" />
-  <xacro:property name="l_rotor_fr_mesh" value="package://meshes/link_rotor_fr.stl" />
-  <xacro:property name="l_rotor_rl_mesh" value="package://meshes/link_rotor_rl.stl" />
-  <xacro:property name="l_rotor_rr_mesh" value="package://meshes/link_rotor_rr.stl" />
+  <xacro:property name="l_rotor_fl_mesh" value="package://enph353-comp-drone/meshes/link_rotor_fl.stl" />
+  <xacro:property name="l_rotor_fr_mesh" value="package://enph353-comp-drone/meshes/link_rotor_fr.stl" />
+  <xacro:property name="l_rotor_rl_mesh" value="package://enph353-comp-drone/meshes/link_rotor_rl.stl" />
+  <xacro:property name="l_rotor_rr_mesh" value="package://enph353-comp-drone/meshes/link_rotor_rr.stl" />
   <xacro:property name="j_rotor_fr_orig_xyz" value="0 0 -0.02" />
   <xacro:property name="j_rotor_fr_orig_rpy" value="3.14159 -0 0" />
@@ -258,5 +258,5 @@
       <origin xyz="-0.000969365 0.000643159 -0.0111761" rpy="0 -0 0" />
       <geometry>
-        <mesh filename="package://meshes/link_drone_body.stl" />
+        <mesh filename="package://enph353-comp-drone/meshes/link_drone_body.stl" />
       </geometry>
       <material name="link_drone_body_material">
@@ -267,5 +267,5 @@
       <origin xyz="-0.000969365 0.000643159 -0.0111761" rpy="0 -0 0" />
       <geometry>
-        <mesh filename="package://meshes/link_drone_body.stl" />
+        <mesh filename="package://enph353-comp-drone/meshes/link_drone_body.stl" />
       </geometry>
     </collision>
@@ -280,5 +280,5 @@
       <origin xyz="-0 -0 0" rpy="3.14159 -0 0" />
       <geometry>
-        <mesh filename="package://meshes/link_imu.stl" />
+        <mesh filename="package://enph353-comp-drone/meshes/link_imu.stl" />
       </geometry>
       <material name="link_imu_material">
@@ -289,5 +289,5 @@
       <origin xyz="-0 -0 0" rpy="3.14159 -0 0" />
       <geometry>
-        <mesh filename="package://meshes/link_imu.stl" />
+        <mesh filename="package://enph353-comp-drone/meshes/link_imu.stl" />
       </geometry>
     </collision>
@@ -302,5 +302,5 @@
       <origin xyz="-0 -0 -0" rpy="1.5708 -0 0" />
       <geometry>
-        <mesh filename="package://meshes/link_camera.stl" />
+        <mesh filename="package://enph353-comp-drone/meshes/link_camera.stl" />
       </geometry>
       <material name="link_camera_material">
@@ -311,5 +311,5 @@
       <origin xyz="-0 -0 -0" rpy="1.5708 -0 0" />
       <geometry>
-        <mesh filename="package://meshes/link_camera.stl" />
+        <mesh filename="package://enph353-comp-drone/meshes/link_camera.stl" />
       </geometry>
     </collision>

Commit message: rotate camera joint to align drone's up with camera's up

File: urdf/drone.urdf.xacro (robot description, xacro)
@@ -323,5 +323,5 @@
   </joint>
   <joint name="joint_camera" type="fixed">
-    <origin xyz="-0.000969365 -0.0193568 -0.00117609" rpy="-1.5708 -0 -0" />
+    <origin xyz="-0.000969365 -0.0193568 -0.00117609" rpy="-1.5708 -0 -1.5708" />
     <parent link="link_drone_body" />
     <child link="link_camera" />

Commit message: change pitch instead of yaw on drone camera joint

File: urdf/drone.urdf.xacro (robot description, xacro)
@@ -323,5 +323,5 @@
   </joint>
   <joint name="joint_camera" type="fixed">
-    <origin xyz="-0.000969365 -0.0193568 -0.00117609" rpy="-1.5708 -0 -1.5708" />
+    <origin xyz="-0.000969365 -0.0193568 -0.00117609" rpy="-1.5708 1.5708 -0" />
     <parent link="link_drone_body" />
     <child link="link_camera" />

Commit message: change roll by 90 degrees

File: urdf/drone.urdf.xacro (robot description, xacro)
@@ -323,5 +323,5 @@
   </joint>
   <joint name="joint_camera" type="fixed">
-    <origin xyz="-0.000969365 -0.0193568 -0.00117609" rpy="-1.5708 1.5708 -0" />
+    <origin xyz="-0.000969365 -0.0193568 -0.00117609" rpy="-1.5708/2 0 -0" />
     <parent link="link_drone_body" />
     <child link="link_camera" />

Commit message: orientation changes

File: urdf/drone.urdf.xacro (robot description, xacro)
@@ -323,5 +323,5 @@
   </joint>
   <joint name="joint_camera" type="fixed">
-    <origin xyz="-0.000969365 -0.0193568 -0.00117609" rpy="-1.5708/2 0 -0" />
+    <origin xyz="-0.000969365 -0.0193568 -0.00117609" rpy="1.5708 0 1.5708" />
     <parent link="link_drone_body" />
     <child link="link_camera" />

Commit message: orientation

File: urdf/drone.urdf.xacro (robot description, xacro)
@@ -323,5 +323,5 @@
   </joint>
   <joint name="joint_camera" type="fixed">
-    <origin xyz="-0.000969365 -0.0193568 -0.00117609" rpy="1.5708 0 1.5708" />
+    <origin xyz="-0.000969365 -0.0193568 -0.00117609" rpy="-3.1416 0 3.1416" />
     <parent link="link_drone_body" />
     <child link="link_camera" />

Commit message: camera joint orientation fixed

File: urdf/drone.urdf.xacro (robot description, xacro)
@@ -323,5 +323,5 @@
   </joint>
   <joint name="joint_camera" type="fixed">
-    <origin xyz="-0.000969365 -0.0193568 -0.00117609" rpy="-3.1416 0 3.1416" />
+    <origin xyz="-0.000969365 -0.0193568 -0.00117609" rpy="-0 0 -1.5708" />
     <parent link="link_drone_body" />
     <child link="link_camera" />

Commit message: first attempt at implementing planar move with drone

File: urdf/drone.urdf.xacro (robot description, xacro)
@@ -25,8 +25,12 @@
   <xacro:property name="l_motor_rl_vis_coll_orig_rpy" value="3.14159 -0 0" />
   <xacro:property name="l_motor_rr_vis_coll_orig_rpy" value="3.14159 -0 0" />
-  <xacro:property name="l_motor_fl_mesh" value="package://enph353-comp-drone/meshes/link_motor_fl.stl" />
-  <xacro:property name="l_motor_fr_mesh" value="package://enph353-comp-drone/meshes/link_motor_fr.stl" />
-  <xacro:property name="l_motor_rl_mesh" value="package://enph353-comp-drone/meshes/link_motor_rl.stl" />
-  <xacro:property name="l_motor_rr_mesh" value="package://enph353-comp-drone/meshes/link_motor_rr.stl" />
+  <xacro:property name="l_motor_fl_mesh"
+    value="package://enph353-comp-drone/meshes/link_motor_fl.stl" />
+  <xacro:property name="l_motor_fr_mesh"
+    value="package://enph353-comp-drone/meshes/link_motor_fr.stl" />
+  <xacro:property name="l_motor_rl_mesh"
+    value="package://enph353-comp-drone/meshes/link_motor_rl.stl" />
+  <xacro:property name="l_motor_rr_mesh"
+    value="package://enph353-comp-drone/meshes/link_motor_rr.stl" />
   <xacro:property name="j_motor_fr_orig_xyz" value="-0.0909694 -0.0893568 -0.0111761" />
   <xacro:property name="j_motor_fr_orig_rpy" value="3.14159 -0 0" />
@@ -69,8 +73,12 @@
   <xacro:property name="l_rotor_rl_vis_coll_orig_rpy" value="0 -0 0" />
   <xacro:property name="l_rotor_rr_vis_coll_orig_rpy" value="0 -0 0" />
-  <xacro:property name="l_rotor_fl_mesh" value="package://enph353-comp-drone/meshes/link_rotor_fl.stl" />
-  <xacro:property name="l_rotor_fr_mesh" value="package://enph353-comp-drone/meshes/link_rotor_fr.stl" />
-  <xacro:property name="l_rotor_rl_mesh" value="package://enph353-comp-drone/meshes/link_rotor_rl.stl" />
-  <xacro:property name="l_rotor_rr_mesh" value="package://enph353-comp-drone/meshes/link_rotor_rr.stl" />
+  <xacro:property name="l_rotor_fl_mesh"
+    value="package://enph353-comp-drone/meshes/link_rotor_fl.stl" />
+  <xacro:property name="l_rotor_fr_mesh"
+    value="package://enph353-comp-drone/meshes/link_rotor_fr.stl" />
+  <xacro:property name="l_rotor_rl_mesh"
+    value="package://enph353-comp-drone/meshes/link_rotor_rl.stl" />
+  <xacro:property name="l_rotor_rr_mesh"
+    value="package://enph353-comp-drone/meshes/link_rotor_rr.stl" />
   <xacro:property name="j_rotor_fr_orig_xyz" value="0 0 -0.02" />
   <xacro:property name="j_rotor_fr_orig_rpy" value="3.14159 -0 0" />
@@ -386,3 +394,12 @@
     </sensor>
   </gazebo>
+  <gazebo>
+    <plugin name="drone_manual_controller" filename="libgazebo_ros_planar_move.so">
+      <commandTopic>cmd_vel</commandTopic>
+      <odometryTopic>odom</odometryTopic>
+      <odometryFrame>odom</odometryFrame>
+      <odometryRate>20.0</odometryRate>
+      <robotBaseFrame>link_drone_body</robotBaseFrame>
+    </plugin>
+  </gazebo>
 </robot>

Commit message: move new meshes in and correct paths in new drone.urdf.xacro

File: urdf/drone.urdf.xacro (robot description, xacro)
@@ -25,8 +25,8 @@
     <xacro:property name="l_motor_rl_vis_coll_orig_rpy" value="3.14159 -0 0" />
     <xacro:property name="l_motor_rr_vis_coll_orig_rpy" value="3.14159 -0 0" />
-    <xacro:property name="l_motor_fl_mesh" value="package://assets/link_motor_fl.stl" />
-    <xacro:property name="l_motor_fr_mesh" value="package://assets/link_motor_fr.stl" />
-    <xacro:property name="l_motor_rl_mesh" value="package://assets/link_motor_rl.stl" />
-    <xacro:property name="l_motor_rr_mesh" value="package://assets/link_motor_rr.stl" />
+    <xacro:property name="l_motor_fl_mesh" value="package://enph353-comp-drone/meshes/link_motor_fl.stl" />
+    <xacro:property name="l_motor_fr_mesh" value="package://enph353-comp-drone/meshes/link_motor_fr.stl" />
+    <xacro:property name="l_motor_rl_mesh" value="package://enph353-comp-drone/meshes/link_motor_rl.stl" />
+    <xacro:property name="l_motor_rr_mesh" value="package://enph353-comp-drone/meshes/link_motor_rr.stl" />
     <xacro:property name="j_motor_fr_orig_xyz" value="0.0897234 -0.0900803 0" />
     <xacro:property name="j_motor_fr_orig_rpy" value="3.14159 -0 1.5708" />
@@ -69,8 +69,8 @@
     <xacro:property name="l_rotor_rl_vis_coll_orig_rpy" value="0 -0 0" />
     <xacro:property name="l_rotor_rr_vis_coll_orig_rpy" value="0 -0 0" />
-    <xacro:property name="l_rotor_fl_mesh" value="package://assets/link_rotor_fl.stl" />
-    <xacro:property name="l_rotor_fr_mesh" value="package://assets/link_rotor_fr.stl" />
-    <xacro:property name="l_rotor_rl_mesh" value="package://assets/link_rotor_rl.stl" />
-    <xacro:property name="l_rotor_rr_mesh" value="package://assets/link_rotor_rr.stl" />
+    <xacro:property name="l_rotor_fl_mesh" value="package://enph353-comp-drone/meshes/link_rotor_fl.stl" />
+    <xacro:property name="l_rotor_fr_mesh" value="package://enph353-comp-drone/meshes/link_rotor_fr.stl" />
+    <xacro:property name="l_rotor_rl_mesh" value="package://enph353-comp-drone/meshes/link_rotor_rl.stl" />
+    <xacro:property name="l_rotor_rr_mesh" value="package://enph353-comp-drone/meshes/link_rotor_rr.stl" />
     <xacro:property name="j_rotor_fr_orig_xyz" value="0 0 -0.02" />
     <xacro:property name="j_rotor_fr_orig_rpy" value="3.14159 -0 1.5708" />
@@ -214,5 +214,5 @@
             <origin xyz="-0.000276567 -8.03059e-05 0" rpy="0 -0 1.5708" />
             <geometry>
-                <mesh filename="package://assets/link_drone_body.stl" />
+                <mesh filename="package://enph353-comp-drone/meshes/link_drone_body.stl" />
             </geometry>
             <material name="link_drone_body_material">
@@ -223,5 +223,5 @@
             <origin xyz="-0.000276567 -8.03059e-05 0" rpy="0 -0 1.5708" />
             <geometry>
-                <mesh filename="package://assets/link_drone_body.stl" />
+                <mesh filename="package://enph353-comp-drone/meshes/link_drone_body.stl" />
             </geometry>
         </collision>
@@ -236,5 +236,5 @@
             <origin xyz="-0 -0 0" rpy="3.14159 -0 0" />
             <geometry>
-                <mesh filename="package://assets/link_imu.stl" />
+                <mesh filename="package://enph353-comp-drone/meshes/link_imu.stl" />
             </geometry>
             <material name="link_imu_material">
@@ -245,5 +245,5 @@
             <origin xyz="-0 -0 0" rpy="3.14159 -0 0" />
             <geometry>
-                <mesh filename="package://assets/link_imu.stl" />
+                <mesh filename="package://enph353-comp-drone/meshes/link_imu.stl" />
             </geometry>
         </collision>
@@ -258,5 +258,5 @@
             <origin xyz="-0 0 0" rpy="1.5708 -0 0" />
             <geometry>
-                <mesh filename="package://assets/link_camera.stl" />
+                <mesh filename="package://enph353-comp-drone/meshes/link_camera.stl" />
             </geometry>
             <material name="link_camera_material">
@@ -267,5 +267,5 @@
             <origin xyz="-0 0 0" rpy="1.5708 -0 0" />
             <geometry>
-                <mesh filename="package://assets/link_camera.stl" />
+                <mesh filename="package://enph353-comp-drone/meshes/link_camera.stl" />
             </geometry>
         </collision>

Commit message: fix camera position on drone

File: urdf/drone.urdf.xacro (robot description, xacro)
@@ -279,5 +279,5 @@
     </joint>
     <joint name="joint_camera" type="fixed">
-        <origin xyz="0.0197234 -8.03059e-05 0.01" rpy="-1.5708 -0 1.5708" />
+        <origin xyz="0.0197234 -8.03059e-05 0.02" rpy="-0 -0 -0" />
         <parent link="link_drone_body" />
         <child link="link_camera" />

Commit message: drone launching into world with keyboard ctrl

File: urdf/drone.urdf.xacro (robot description, xacro)
@@ -25,8 +25,8 @@
     <xacro:property name="l_motor_rl_vis_coll_orig_rpy" value="3.14159 -0 0" />
     <xacro:property name="l_motor_rr_vis_coll_orig_rpy" value="3.14159 -0 0" />
-    <xacro:property name="l_motor_fl_mesh" value="package://enph353-comp-drone/meshes/link_motor_fl.stl" />
-    <xacro:property name="l_motor_fr_mesh" value="package://enph353-comp-drone/meshes/link_motor_fr.stl" />
-    <xacro:property name="l_motor_rl_mesh" value="package://enph353-comp-drone/meshes/link_motor_rl.stl" />
-    <xacro:property name="l_motor_rr_mesh" value="package://enph353-comp-drone/meshes/link_motor_rr.stl" />
+    <xacro:property name="l_motor_fl_mesh" value="package://drone_desc/meshes/link_motor_fl.stl" />
+    <xacro:property name="l_motor_fr_mesh" value="package://drone_desc/meshes/link_motor_fr.stl" />
+    <xacro:property name="l_motor_rl_mesh" value="package://drone_desc/meshes/link_motor_rl.stl" />
+    <xacro:property name="l_motor_rr_mesh" value="package://drone_desc/meshes/link_motor_rr.stl" />
     <xacro:property name="j_motor_fr_orig_xyz" value="0.0897234 -0.0900803 0" />
     <xacro:property name="j_motor_fr_orig_rpy" value="3.14159 -0 1.5708" />
@@ -69,8 +69,8 @@
     <xacro:property name="l_rotor_rl_vis_coll_orig_rpy" value="0 -0 0" />
     <xacro:property name="l_rotor_rr_vis_coll_orig_rpy" value="0 -0 0" />
-    <xacro:property name="l_rotor_fl_mesh" value="package://enph353-comp-drone/meshes/link_rotor_fl.stl" />
-    <xacro:property name="l_rotor_fr_mesh" value="package://enph353-comp-drone/meshes/link_rotor_fr.stl" />
-    <xacro:property name="l_rotor_rl_mesh" value="package://enph353-comp-drone/meshes/link_rotor_rl.stl" />
-    <xacro:property name="l_rotor_rr_mesh" value="package://enph353-comp-drone/meshes/link_rotor_rr.stl" />
+    <xacro:property name="l_rotor_fl_mesh" value="package://drone_desc/meshes/link_rotor_fl.stl" />
+    <xacro:property name="l_rotor_fr_mesh" value="package://drone_desc/meshes/link_rotor_fr.stl" />
+    <xacro:property name="l_rotor_rl_mesh" value="package://drone_desc/meshes/link_rotor_rl.stl" />
+    <xacro:property name="l_rotor_rr_mesh" value="package://drone_desc/meshes/link_rotor_rr.stl" />
     <xacro:property name="j_rotor_fr_orig_xyz" value="0 0 -0.02" />
     <xacro:property name="j_rotor_fr_orig_rpy" value="3.14159 -0 1.5708" />
@@ -214,5 +214,5 @@
             <origin xyz="-0.000276567 -8.03059e-05 0" rpy="0 -0 1.5708" />
             <geometry>
-                <mesh filename="package://enph353-comp-drone/meshes/link_drone_body.stl" />
+                <mesh filename="package://drone_desc/meshes/link_drone_body.stl" />
             </geometry>
             <material name="link_drone_body_material">
@@ -223,5 +223,5 @@
             <origin xyz="-0.000276567 -8.03059e-05 0" rpy="0 -0 1.5708" />
             <geometry>
-                <mesh filename="package://enph353-comp-drone/meshes/link_drone_body.stl" />
+                <mesh filename="package://drone_desc/meshes/link_drone_body.stl" />
             </geometry>
         </collision>
@@ -236,5 +236,5 @@
             <origin xyz="-0 -0 0" rpy="3.14159 -0 0" />
             <geometry>
-                <mesh filename="package://enph353-comp-drone/meshes/link_imu.stl" />
+                <mesh filename="package://drone_desc/meshes/link_imu.stl" />
             </geometry>
             <material name="link_imu_material">
@@ -245,5 +245,5 @@
             <origin xyz="-0 -0 0" rpy="3.14159 -0 0" />
             <geometry>
-                <mesh filename="package://enph353-comp-drone/meshes/link_imu.stl" />
+                <mesh filename="package://drone_desc/meshes/link_imu.stl" />
             </geometry>
         </collision>
@@ -258,5 +258,5 @@
             <origin xyz="-0 0 0" rpy="1.5708 -0 0" />
             <geometry>
-                <mesh filename="package://enph353-comp-drone/meshes/link_camera.stl" />
+                <mesh filename="package://drone_desc/meshes/link_camera.stl" />
             </geometry>
             <material name="link_camera_material">
@@ -267,5 +267,5 @@
             <origin xyz="-0 0 0" rpy="1.5708 -0 0" />
             <geometry>
-                <mesh filename="package://enph353-comp-drone/meshes/link_camera.stl" />
+                <mesh filename="package://drone_desc/meshes/link_camera.stl" />
             </geometry>
         </collision>

File: urdf/old_drone.urdf.xacro (robot description, xacro)
@@ -1,4 +1,4 @@
 <?xml version='1.0' encoding='utf-8'?>
-<robot xmlns:xacro="http://www.ros.org/wiki/xacro" name="enph353-comp-drone">
+<robot xmlns:xacro="http://www.ros.org/wiki/xacro" name="drone_desc">
   <xacro:property name="l_motor_fl_inert_orig_xyz" value="0 -0 -0.0101836" />
   <xacro:property name="l_motor_fr_inert_orig_xyz" value="0 -0 -0.0101836" />
@@ -26,11 +26,11 @@
   <xacro:property name="l_motor_rr_vis_coll_orig_rpy" value="3.14159 -0 0" />
   <xacro:property name="l_motor_fl_mesh"
-    value="package://enph353-comp-drone/meshes/link_motor_fl.stl" />
+    value="package://drone_desc/meshes/link_motor_fl.stl" />
   <xacro:property name="l_motor_fr_mesh"
-    value="package://enph353-comp-drone/meshes/link_motor_fr.stl" />
+    value="package://drone_desc/meshes/link_motor_fr.stl" />
   <xacro:property name="l_motor_rl_mesh"
-    value="package://enph353-comp-drone/meshes/link_motor_rl.stl" />
+    value="package://drone_desc/meshes/link_motor_rl.stl" />
   <xacro:property name="l_motor_rr_mesh"
-    value="package://enph353-comp-drone/meshes/link_motor_rr.stl" />
+    value="package://drone_desc/meshes/link_motor_rr.stl" />
   <xacro:property name="j_motor_fr_orig_xyz" value="-0.0909694 -0.0893568 -0.0111761" />
   <xacro:property name="j_motor_fr_orig_rpy" value="3.14159 -0 0" />
@@ -74,11 +74,11 @@
   <xacro:property name="l_rotor_rr_vis_coll_orig_rpy" value="0 -0 0" />
   <xacro:property name="l_rotor_fl_mesh"
-    value="package://enph353-comp-drone/meshes/link_rotor_fl.stl" />
+    value="package://drone_desc/meshes/link_rotor_fl.stl" />
   <xacro:property name="l_rotor_fr_mesh"
-    value="package://enph353-comp-drone/meshes/link_rotor_fr.stl" />
+    value="package://drone_desc/meshes/link_rotor_fr.stl" />
   <xacro:property name="l_rotor_rl_mesh"
-    value="package://enph353-comp-drone/meshes/link_rotor_rl.stl" />
+    value="package://drone_desc/meshes/link_rotor_rl.stl" />
   <xacro:property name="l_rotor_rr_mesh"
-    value="package://enph353-comp-drone/meshes/link_rotor_rr.stl" />
+    value="package://drone_desc/meshes/link_rotor_rr.stl" />
   <xacro:property name="j_rotor_fr_orig_xyz" value="0 0 -0.02" />
   <xacro:property name="j_rotor_fr_orig_rpy" value="3.14159 -0 0" />
@@ -266,5 +266,5 @@
       <origin xyz="-0.000969365 0.000643159 -0.0111761" rpy="0 -0 0" />
       <geometry>
-        <mesh filename="package://enph353-comp-drone/meshes/link_drone_body.stl" />
+        <mesh filename="package://drone_desc/meshes/link_drone_body.stl" />
       </geometry>
       <material name="link_drone_body_material">
@@ -275,5 +275,5 @@
       <origin xyz="-0.000969365 0.000643159 -0.0111761" rpy="0 -0 0" />
       <geometry>
-        <mesh filename="package://enph353-comp-drone/meshes/link_drone_body.stl" />
+        <mesh filename="package://drone_desc/meshes/link_drone_body.stl" />
       </geometry>
     </collision>
@@ -288,5 +288,5 @@
       <origin xyz="-0 -0 0" rpy="3.14159 -0 0" />
       <geometry>
-        <mesh filename="package://enph353-comp-drone/meshes/link_imu.stl" />
+        <mesh filename="package://drone_desc/meshes/link_imu.stl" />
       </geometry>
       <material name="link_imu_material">
@@ -297,5 +297,5 @@
       <origin xyz="-0 -0 0" rpy="3.14159 -0 0" />
       <geometry>
-        <mesh filename="package://enph353-comp-drone/meshes/link_imu.stl" />
+        <mesh filename="package://drone_desc/meshes/link_imu.stl" />
       </geometry>
     </collision>
@@ -310,5 +310,5 @@
       <origin xyz="-0 -0 -0" rpy="1.5708 -0 0" />
       <geometry>
-        <mesh filename="package://enph353-comp-drone/meshes/link_camera.stl" />
+        <mesh filename="package://drone_desc/meshes/link_camera.stl" />
       </geometry>
       <material name="link_camera_material">
@@ -319,5 +319,5 @@
       <origin xyz="-0 -0 -0" rpy="1.5708 -0 0" />
       <geometry>
-        <mesh filename="package://enph353-comp-drone/meshes/link_camera.stl" />
+        <mesh filename="package://drone_desc/meshes/link_camera.stl" />
       </geometry>
     </collision>
