Commit message: added new camera to the bottom of the drone facing downward

File: urdf/drone.urdf.xacro (robot description, xacro)
@@ -276,4 +276,26 @@
         </collision>
     </link>
+    <link name="link_down_camera">
+        <inertial>
+            <origin xyz="-0 0 -0.0" rpy="0 0 0" />
+            <mass value="0.01" />
+            <inertia ixx="4.16667e-07" ixy="0" ixz="0" iyy="4.16667e-07" iyz="0" izz="6.66667e-07" />
+        </inertial>
+        <visual>
+            <origin xyz="-0 0 0" rpy="1.5708 -0 0" />
+            <geometry>
+                <mesh filename="package://drone_desc/meshes/link_camera.stl" />
+            </geometry>
+            <material name="link_camera_material">
+                <color rgba="0 0 1 1" />
+            </material>
+        </visual>
+        <collision>
+            <origin xyz="-0 0 0" rpy="1.5708 -0 0" />
+            <geometry>
+                <mesh filename="package://drone_desc/meshes/link_camera.stl" />
+            </geometry>
+        </collision>
+    </link>
     <joint name="joint_imu" type="fixed">
         <origin xyz="-0.000276567 -8.03059e-05 0.005" rpy="3.14159 -0 1.5708" />
@@ -287,6 +309,9 @@
         <parent link="link_drone_body" />
         <child link="link_camera" />
-        <axis xyz="0 0 1" />
-        <limit effort="10" velocity="10" />
+    </joint>
+    <joint name="joint_down_camera" type="fixed">
+        <origin xyz="0.0 0.0 -0.01" rpy="-0 1.5708 -0" />
+        <parent link="link_drone_body" />
+        <child link="link_down_camera" />
     </joint>
     <!-- End of Extra Links and Joints -->
@@ -315,5 +340,5 @@
         <sensor type="camera" name="camera1">
             <update_rate>30.0</update_rate>
-            <camera name="head">
+            <camera name="front_cam">
                 <horizontal_fov>1.3962634</horizontal_fov>
                 <image>
@@ -332,5 +357,5 @@
                 </noise>
             </camera>
-            <plugin name="camera_controller" filename="libgazebo_ros_camera.so">
+            <plugin name="front_cam" filename="libgazebo_ros_camera.so">
                 <alwaysOn>true</alwaysOn>
                 <updateRate>0.0</updateRate>
@@ -348,5 +373,41 @@
         </sensor>
     </gazebo>
-    <!-- plugin for robot to fly by plane-->
+    <gazebo reference="link_down_camera">
+        <sensor type="camera" name="camera2">
+            <update_rate>30.0</update_rate>
+            <camera name="down_cam">
+                <horizontal_fov>1.3962634</horizontal_fov>
+                <image>
+                    <width>800</width>
+                    <height>800</height>
+                    <format>R8G8B8</format>
+                </image>
+                <clip>
+                    <near>0.02</near>
+                    <far>300</far>
+                </clip>
+                <noise>
+                    <type>gaussian</type>
+                    <mean>0.0</mean>
+                    <stddev>0.007</stddev>
+                </noise>
+            </camera>
+            <plugin name="down_cam" filename="libgazebo_ros_camera.so">
+                <alwaysOn>true</alwaysOn>
+                <updateRate>0.0</updateRate>
+                <cameraName>camera2</cameraName>
+                <imageTopicName>image_raw</imageTopicName>
+                <cameraInfoTopicName>camera_info</cameraInfoTopicName>
+                <frameName>link_down_camera</frameName>
+                <hackBaseline>0.07</hackBaseline>
+                <distortionK1>0.0</distortionK1>
+                <distortionK2>0.0</distortionK2>
+                <distortionK3>0.0</distortionK3>
+                <distortionT1>0.0</distortionT1>
+                <distortionT2>0.0</distortionT2>
+            </plugin>
+        </sensor>
+    </gazebo>
+    <!-- plugin for robot to fly by plane -->
     <gazebo>
         <plugin name="drone_planar_mov" filename="libgazebo_ros_planar_move.so">

Commit message: added down laser to robot-not tested

File: urdf/drone.urdf.xacro (robot description, xacro)
@@ -254,4 +254,5 @@
         </collision>
     </link>
+    <!-- LINK - CAMERA - FRONTWARD FACING -->
     <link name="link_camera">
         <inertial>
@@ -276,5 +277,29 @@
         </collision>
     </link>
+    <!-- LINK - CAMERA - DOWNWARD FACING -->
     <link name="link_down_camera">
+        <inertial>
+            <origin xyz="-0 0 -0.0" rpy="0 0 0" />
+            <mass value="0.01" />
+            <inertia ixx="4.16667e-07" ixy="0" ixz="0" iyy="4.16667e-07" iyz="0" izz="6.66667e-07" />
+        </inertial>
+        <visual>
+            <origin xyz="-0 0 0" rpy="1.5708 -0 0" />
+            <geometry>
+                <mesh filename="package://drone_desc/meshes/link_camera.stl" />
+            </geometry>
+            <material name="link_camera_material">
+                <color rgba="0 0 1 1" />
+            </material>
+        </visual>
+        <collision>
+            <origin xyz="-0 0 0" rpy="1.5708 -0 0" />
+            <geometry>
+                <mesh filename="package://drone_desc/meshes/link_camera.stl" />
+            </geometry>
+        </collision>
+    </link>
+    <!-- LINK - LASER - DOWNWARD FACING (just use same linktype as camera for now)-->
+    <link name="link_down_laser">
         <inertial>
             <origin xyz="-0 0 -0.0" rpy="0 0 0" />
@@ -314,4 +339,9 @@
         <parent link="link_drone_body" />
         <child link="link_down_camera" />
+    </joint>
+    <joint name="joint_down_laser" type="fixed">
+        <origin xyz="-0.01 0.0 -0.01" rpy="-0 1.5708 -0" />
+        <parent link="link_drone_body" />
+        <child link="link_down_laser" />
     </joint>
     <!-- End of Extra Links and Joints -->
@@ -409,4 +439,40 @@
         </sensor>
     </gazebo>
+    <!-- DOWN LASER -->
+    <gazebo reference="link_down_laser">
+        <sensor type="ray" name="head_hokuyo_sensor">
+        <pose>0 0 0 0 0 0</pose>
+        <visualize>true</visualize>
+        <update_rate>40</update_rate>
+        <ray>
+            <scan>
+            <horizontal>
+                <samples>720</samples>
+                <resolution>1</resolution>
+                <min_angle>-1.570796</min_angle>
+                <max_angle>1.570796</max_angle>
+            </horizontal>
+            </scan>
+            <range>
+            <min>0.10</min>
+            <max>30.0</max>
+            <resolution>0.01</resolution>
+            </range>
+            <noise>
+            <type>gaussian</type>
+            <!-- Noise parameters based on published spec for Hokuyo laser
+                achieving "+-30mm" accuracy at range < 10m.  A mean of 0.0m and
+                stddev of 0.01m will put 99.7% of samples within 0.03m of the true
+                reading. -->
+            <mean>0.0</mean>
+            <stddev>0.01</stddev>
+            </noise>
+        </ray>
+        <plugin name="gazebo_ros_head_hokuyo_controller" filename="libgazebo_ros_laser.so">
+            <topicName>/rrbot/laser/scan</topicName>
+            <frameName>hokuyo_link</frameName>
+        </plugin>
+        </sensor>
+    </gazebo>
     <!-- plugin for robot to fly by plane -->
     <gazebo>

Commit message: distanced down laser and down camera and renamed laser topic

File: urdf/drone.urdf.xacro (robot description, xacro)
@@ -336,5 +336,5 @@
     </joint>
     <joint name="joint_down_camera" type="fixed">
-        <origin xyz="0.0 0.0 -0.01" rpy="-0 1.5708 -0" />
+        <origin xyz="0.01 0.0 -0.01" rpy="-0 1.5708 -0" />
         <parent link="link_drone_body" />
         <child link="link_down_camera" />
@@ -470,5 +470,5 @@
         </ray>
         <plugin name="gazebo_ros_head_hokuyo_controller" filename="libgazebo_ros_laser.so">
-            <topicName>/rrbot/laser/scan</topicName>
+            <topicName>down_laser/scan</topicName>
             <frameName>hokuyo_link</frameName>
         </plugin>

Commit message: added stabilization prototype ot drone_cmd_bridge, should be moved. Reoriented imu for perfect alignment with drone

File: urdf/drone.urdf.xacro (robot description, xacro)
@@ -324,9 +324,7 @@
     </link>
     <joint name="joint_imu" type="fixed">
-        <origin xyz="-0.000276567 -8.03059e-05 0.005" rpy="3.14159 -0 1.5708" />
+        <origin xyz="0 0 0.005" rpy="0 0 0" />
         <parent link="link_drone_body" />
         <child link="link_imu" />
-        <axis xyz="0 0 1" />
-        <limit effort="10" velocity="10" />
     </joint>
     <joint name="joint_camera" type="fixed">
@@ -476,9 +474,9 @@
         </sensor>
     </gazebo>
-    <!-- plugin for robot to fly plane -->
+    <!-- plugin for robot to fly -->
     <gazebo>
         <plugin name="drone_mov" filename="libgazebo_ros_force.so">
-            <!-- <robotNamespace>/thing</robotNamespace> -->
-            <bodyName>link_drone_body</bodyName>
+            <robotNamespace>$(arg name)</robotNamespace>
+            <bodyName>$(arg name)::link_drone_body</bodyName>
             <topicName>cmd_force</topicName>
         </plugin>

Commit message: add little stands and modify cam

File: urdf/drone.urdf.xacro (robot description, xacro)
@@ -211,5 +211,5 @@
     <link name="link_drone_body">
         <inertial>
-            <origin xyz="-0.000304819 -3.77332e-05 0.00999998" rpy="0 0 0" />
+            <origin xyz="0.0 0.0 0.01" rpy="0 0 0" />
             <mass value="0.27585" />
             <inertia ixx="0.000944175" ixy="8.5525e-07" ixz="-1.878e-09" iyy="0.000942851"
@@ -280,5 +280,5 @@
     <link name="link_down_camera">
         <inertial>
-            <origin xyz="-0 0 -0.0" rpy="0 0 0" />
+            <origin xyz="-0 0 -0.005" rpy="0 0 0" />
             <mass value="0.01" />
             <inertia ixx="4.16667e-07" ixy="0" ixz="0" iyy="4.16667e-07" iyz="0" izz="6.66667e-07" />
@@ -303,5 +303,5 @@
     <link name="link_down_laser">
         <inertial>
-            <origin xyz="-0 0 -0.0" rpy="0 0 0" />
+            <origin xyz="-0 0 -0.005" rpy="0 0 0" />
             <mass value="0.01" />
             <inertia ixx="4.16667e-07" ixy="0" ixz="0" iyy="4.16667e-07" iyz="0" izz="6.66667e-07" />
@@ -323,4 +323,92 @@
         </collision>
     </link>
+    <link name="link_stand1">
+        <inertial>
+            <origin xyz="-0.00 -0.00 -0.01" rpy="0 0 0" />
+            <mass value="0.01" />
+            <inertia ixx="4.16667e-07" ixy="0" ixz="0" iyy="4.16667e-07" iyz="0" izz="6.66667e-07" />
+        </inertial>
+        <visual>
+            <origin xyz="-0 0 0" rpy="1.5708 -0 0" />
+            <geometry>
+                <mesh filename="package://drone_desc/meshes/link_camera.stl" />
+            </geometry>
+            <material name="link_camera_material">
+                <color rgba="0 0 1 1" />
+            </material>
+        </visual>
+        <collision>
+            <origin xyz="-0 0 0" rpy="1.5708 -0 0" />
+            <geometry>
+                <mesh filename="package://drone_desc/meshes/link_camera.stl" />
+            </geometry>
+        </collision>
+    </link>
+    <link name="link_stand2">
+        <inertial>
+            <origin xyz="-0.00 -0.00 -0.01" rpy="0 0 0" />
+            <mass value="0.01" />
+            <inertia ixx="4.16667e-07" ixy="0" ixz="0" iyy="4.16667e-07" iyz="0" izz="6.66667e-07" />
+        </inertial>
+        <visual>
+            <origin xyz="-0 0 0" rpy="1.5708 -0 0" />
+            <geometry>
+                <mesh filename="package://drone_desc/meshes/link_camera.stl" />
+            </geometry>
+            <material name="link_camera_material">
+                <color rgba="0 0 1 1" />
+            </material>
+        </visual>
+        <collision>
+            <origin xyz="-0 0 0" rpy="1.5708 -0 0" />
+            <geometry>
+                <mesh filename="package://drone_desc/meshes/link_camera.stl" />
+            </geometry>
+        </collision>
+    </link>
+    <link name="link_stand3">
+        <inertial>
+            <origin xyz="-0.00 -0.00 -0.01" rpy="0 0 0" />
+            <mass value="0.01" />
+            <inertia ixx="4.16667e-07" ixy="0" ixz="0" iyy="4.16667e-07" iyz="0" izz="6.66667e-07" />
+        </inertial>
+        <visual>
+            <origin xyz="-0 0 0" rpy="1.5708 -0 0" />
+            <geometry>
+                <mesh filename="package://drone_desc/meshes/link_camera.stl" />
+            </geometry>
+            <material name="link_camera_material">
+                <color rgba="0 0 1 1" />
+            </material>
+        </visual>
+        <collision>
+            <origin xyz="-0 0 0" rpy="1.5708 -0 0" />
+            <geometry>
+                <mesh filename="package://drone_desc/meshes/link_camera.stl" />
+            </geometry>
+        </collision>
+    </link>
+    <link name="link_stand4">
+        <inertial>
+            <origin xyz="-0.00 -0.00 -0.01" rpy="0 0 0" />
+            <mass value="0.01" />
+            <inertia ixx="4.16667e-07" ixy="0" ixz="0" iyy="4.16667e-07" iyz="0" izz="6.66667e-07" />
+        </inertial>
+        <visual>
+            <origin xyz="-0 0 0" rpy="1.5708 -0 0" />
+            <geometry>
+                <mesh filename="package://drone_desc/meshes/link_camera.stl" />
+            </geometry>
+            <material name="link_camera_material">
+                <color rgba="0 0 1 1" />
+            </material>
+        </visual>
+        <collision>
+            <origin xyz="-0 0 0" rpy="1.5708 -0 0" />
+            <geometry>
+                <mesh filename="package://drone_desc/meshes/link_camera.stl" />
+            </geometry>
+        </collision>
+    </link>
     <joint name="joint_imu" type="fixed">
         <origin xyz="0 0 0.005" rpy="0 0 0" />
@@ -329,17 +417,38 @@
     </joint>
     <joint name="joint_camera" type="fixed">
-        <origin xyz="0.0197234 -8.03059e-05 0.02" rpy="-0 -0 -0" />
+        <origin xyz="0.0197234 -0.0 0.02" rpy="-0 -0 -0" />
         <parent link="link_drone_body" />
         <child link="link_camera" />
     </joint>
     <joint name="joint_down_camera" type="fixed">
-        <origin xyz="0.01 0.0 -0.01" rpy="-0 1.5708 -0" />
+        <origin xyz="0.01 0.0 0.005" rpy="-0 1.5708 -0" />
         <parent link="link_drone_body" />
         <child link="link_down_camera" />
     </joint>
     <joint name="joint_down_laser" type="fixed">
-        <origin xyz="-0.01 0.0 -0.01" rpy="-0 1.5708 -0" />
+        <origin xyz="-0.01 0.0 0.005" rpy="-0 1.5708 -0" />
         <parent link="link_drone_body" />
         <child link="link_down_laser" />
+    </joint>
+    <!-- DRONE STAND JOINTS -->
+    <joint name="joint_stand1" type="fixed">
+        <origin xyz="0.03 0.03 -0.005" rpy="-0 1.5708 -0" />
+        <parent link="link_drone_body" />
+        <child link="link_stand1" />
+    </joint>
+    <joint name="joint_stand2" type="fixed">
+        <origin xyz="0.03 -0.03 -0.005" rpy="-0 1.5708 -0" />
+        <parent link="link_drone_body" />
+        <child link="link_stand2" />
+    </joint>
+    <joint name="joint_stand3" type="fixed">
+        <origin xyz="-0.03 0.03 -0.005" rpy="-0 1.5708 -0" />
+        <parent link="link_drone_body" />
+        <child link="link_stand3" />
+    </joint>
+    <joint name="joint_stand4" type="fixed">
+        <origin xyz="-0.03 -0.03 -0.005" rpy="-0 1.5708 -0" />
+        <parent link="link_drone_body" />
+        <child link="link_stand4" />
     </joint>
     <!-- End of Extra Links and Joints -->
@@ -355,5 +464,5 @@
                 <topicName>imu</topicName> <!-- inherits namespace, doesn't need  -->
                 <bodyName>link_imu</bodyName>
-                <updateRateHZ>100.0</updateRateHZ>
+                <updateRateHZ>30.0</updateRateHZ>
                 <gaussianNoise>0.0</gaussianNoise>
                 <xyzOffset>0 0 0</xyzOffset>
@@ -443,5 +552,5 @@
         <pose>0 0 0 0 0 0</pose>
         <visualize>true</visualize>
-        <update_rate>40</update_rate>
+        <update_rate>30.0</update_rate>
         <ray>
             <scan>
@@ -455,5 +564,5 @@
             <range>
             <min>0.10</min>
-            <max>30.0</max>
+            <max>100.0</max>
             <resolution>0.01</resolution>
             </range>
