Commit message: removed obligation to launch drone_cmd_bridge from drone_spawn.launch. That is now with individual control mode launchers

File: urdf/drone.urdf.xacro (robot description, xacro)
@@ -232,4 +232,135 @@
         </collision>
     </link>
+    <!-- DRONE BODY NEON ORANGE -->
+    <gazebo reference="link_drone_body">
+        <visual>
+            <material>
+                <ambient>1 0.5 0 1</ambient>
+                <diffuse>1 0.5 0 1</diffuse>
+                <specular>0.5 0.5 0.5 1</specular>
+                <emissive>0.6 0.3 0 1</emissive>
+            </material>
+        </visual>
+    </gazebo>
+    <gazebo reference="link_rotor_fr">
+        <visual>
+            <material>
+                <ambient>1 0.5 0 1</ambient>
+                <diffuse>1 0.5 0 1</diffuse>
+                <specular>0.5 0.5 0.5 1</specular>
+                <emissive>0.6 0.3 0 1</emissive>
+            </material>
+        </visual>
+    </gazebo>
+    <gazebo reference="link_rotor_fl">
+        <visual>
+            <material>
+                <ambient>1 0.5 0 1</ambient>
+                <diffuse>1 0.5 0 1</diffuse>
+                <specular>0.5 0.5 0.5 1</specular>
+                <emissive>0.6 0.3 0 1</emissive>
+            </material>
+        </visual>
+    </gazebo>
+    <gazebo reference="link_rotor_rl">
+        <visual>
+            <material>
+                <ambient>1 0.5 0 1</ambient>
+                <diffuse>1 0.5 0 1</diffuse>
+                <specular>0.5 0.5 0.5 1</specular>
+                <emissive>0.6 0.3 0 1</emissive>
+            </material>
+        </visual>
+    </gazebo><gazebo reference="link_rotor_rr">
+        <visual>
+            <material>
+                <ambient>1 0.5 0 1</ambient>
+                <diffuse>1 0.5 0 1</diffuse>
+                <specular>0.5 0.5 0.5 1</specular>
+                <emissive>0.6 0.3 0 1</emissive>
+            </material>
+        </visual>
+    </gazebo>
+    <gazebo reference="link_motor_fr">
+        <visual>
+            <material>
+                <ambient>1 0.5 0 1</ambient>
+                <diffuse>1 0.5 0 1</diffuse>
+                <specular>0.5 0.5 0.5 1</specular>
+                <emissive>0.6 0.3 0 1</emissive>
+            </material>
+        </visual>
+    </gazebo>
+    <gazebo reference="link_motor_fl">
+        <visual>
+            <material>
+                <ambient>1 0.5 0 1</ambient>
+                <diffuse>1 0.5 0 1</diffuse>
+                <specular>0.5 0.5 0.5 1</specular>
+                <emissive>0.6 0.3 0 1</emissive>
+            </material>
+        </visual>
+    </gazebo>
+    <gazebo reference="link_motor_rl">
+        <visual>
+            <material>
+                <ambient>1 0.5 0 1</ambient>
+                <diffuse>1 0.5 0 1</diffuse>
+                <specular>0.5 0.5 0.5 1</specular>
+                <emissive>0.6 0.3 0 1</emissive>
+            </material>
+        </visual>
+    </gazebo>
+    <gazebo reference="link_motor_rr">
+        <visual>
+            <material>
+                <ambient>1 0.5 0 1</ambient>
+                <diffuse>1 0.5 0 1</diffuse>
+                <specular>0.5 0.5 0.5 1</specular>
+                <emissive>0.6 0.3 0 1</emissive>
+            </material>
+        </visual>
+    </gazebo>
+    <gazebo reference="link_front_camera">
+        <visual>
+            <material>
+                <ambient>1 0.5 0 1</ambient>
+                <diffuse>1 0.5 0 1</diffuse>
+                <specular>0.5 0.5 0.5 1</specular>
+                <emissive>0.6 0.3 0 1</emissive>
+            </material>
+        </visual>
+    </gazebo>
+    <gazebo reference="link_back_camera">
+        <visual>
+            <material>
+                <ambient>1 0.5 0 1</ambient>
+                <diffuse>1 0.5 0 1</diffuse>
+                <specular>0.5 0.5 0.5 1</specular>
+                <emissive>0.6 0.3 0 1</emissive>
+            </material>
+        </visual>
+    </gazebo>
+    <gazebo reference="link_right_camera">
+        <visual>
+            <material>
+                <ambient>1 0.5 0 1</ambient>
+                <diffuse>1 0.5 0 1</diffuse>
+                <specular>0.5 0.5 0.5 1</specular>
+                <emissive>0.6 0.3 0 1</emissive>
+            </material>
+        </visual>
+    </gazebo>
+    <gazebo reference="link_left_camera">
+        <visual>
+            <material>
+                <ambient>1 0.5 0 1</ambient>
+                <diffuse>1 0.5 0 1</diffuse>
+                <specular>0.5 0.5 0.5 1</specular>
+                <emissive>0.6 0.3 0 1</emissive>
+            </material>
+        </visual>
+    </gazebo>
+    <!-- IMU LINK -->
     <link name="link_imu">
         <inertial>
@@ -255,5 +386,5 @@
     </link>
     <!-- LINK - CAMERA - FRONTWARD FACING -->
-    <link name="link_camera">
+    <link name="link_front_camera">
         <inertial>
             <origin xyz="-0 0 -0.005" rpy="0 0 0" />
@@ -277,4 +408,73 @@
         </collision>
     </link>
+    <!-- LINK - CAMERA - LEFTWARD FACING -->
+    <link name="link_left_camera">
+        <inertial>
+            <origin xyz="-0 0 -0.005" rpy="0 0 0" />
+            <mass value="0.01" />
+            <inertia ixx="4.16667e-07" ixy="0" ixz="0" iyy="4.16667e-07" iyz="0" izz="6.66667e-07" />
+        </inertial>
+        <visual>
+            <origin xyz="-0 0 0" rpy="1.5708 -0 0" />
+            <geometry>
+                <mesh filename="package://drone_desc/meshes/link_camera.stl" />
+            </geometry>
+            <material name="link_camera_material">
+                <color rgba="0 0 1 1" />
+            </material>
+        </visual>
+        <collision>
+            <origin xyz="-0 0 0" rpy="1.5708 -0 0" />
+            <geometry>
+                <mesh filename="package://drone_desc/meshes/link_camera.stl" />
+            </geometry>
+        </collision>
+    </link>
+    <!-- LINK - CAMERA - RIGHTWARD FACING -->
+    <link name="link_right_camera">
+        <inertial>
+            <origin xyz="-0 0 -0.005" rpy="0 0 0" />
+            <mass value="0.01" />
+            <inertia ixx="4.16667e-07" ixy="0" ixz="0" iyy="4.16667e-07" iyz="0" izz="6.66667e-07" />
+        </inertial>
+        <visual>
+            <origin xyz="-0 0 0" rpy="1.5708 -0 0" />
+            <geometry>
+                <mesh filename="package://drone_desc/meshes/link_camera.stl" />
+            </geometry>
+            <material name="link_camera_material">
+                <color rgba="0 0 1 1" />
+            </material>
+        </visual>
+        <collision>
+            <origin xyz="-0 0 0" rpy="1.5708 -0 0" />
+            <geometry>
+                <mesh filename="package://drone_desc/meshes/link_camera.stl" />
+            </geometry>
+        </collision>
+    </link>
+    <!-- LINK - CAMERA - BACKWARD FACING -->
+    <link name="link_back_camera">
+        <inertial>
+            <origin xyz="-0 0 -0.005" rpy="0 0 0" />
+            <mass value="0.01" />
+            <inertia ixx="4.16667e-07" ixy="0" ixz="0" iyy="4.16667e-07" iyz="0" izz="6.66667e-07" />
+        </inertial>
+        <visual>
+            <origin xyz="-0 0 0" rpy="1.5708 -0 0" />
+            <geometry>
+                <mesh filename="package://drone_desc/meshes/link_camera.stl" />
+            </geometry>
+            <material name="link_camera_material">
+                <color rgba="0 0 1 1" />
+            </material>
+        </visual>
+        <collision>
+            <origin xyz="-0 0 0" rpy="1.5708 -0 0" />
+            <geometry>
+                <mesh filename="package://drone_desc/meshes/link_camera.stl" />
+            </geometry>
+        </collision>
+    </link>
     <!-- LINK - CAMERA - DOWNWARD FACING -->
     <link name="link_down_camera">
@@ -301,5 +501,5 @@
     </link>
     <!-- LINK - LASER - DOWNWARD FACING (just use same linktype as camera for now)-->
-    <link name="link_down_laser">
+    <link name="link_down_depth">
         <inertial>
             <origin xyz="-0 0 -0.005" rpy="0 0 0" />
@@ -323,4 +523,5 @@
         </collision>
     </link>
+    <!-- STAND FOR DRONE TO REST ON -->
     <link name="link_stand1">
         <inertial>
@@ -416,8 +617,23 @@
         <child link="link_imu" />
     </joint>
-    <joint name="joint_camera" type="fixed">
+    <joint name="joint_front_camera" type="fixed">
         <origin xyz="0.0197234 -0.0 0.02" rpy="-0 -0 -0" />
         <parent link="link_drone_body" />
-        <child link="link_camera" />
+        <child link="link_front_camera" />
+    </joint>
+    <joint name="joint_left_camera" type="fixed">
+        <origin xyz="0.0 0.0197234 0.02" rpy="-0 -0 1.570796" />
+        <parent link="link_drone_body" />
+        <child link="link_left_camera" />
+    </joint>
+    <joint name="joint_right_camera" type="fixed">
+        <origin xyz="0.0 -0.0197234 0.02" rpy="-0 -0 -1.570796" />
+        <parent link="link_drone_body" />
+        <child link="link_right_camera" />
+    </joint>
+    <joint name="joint_back_camera" type="fixed">
+        <origin xyz="-0.0197234 -0.0 0.02" rpy="-0 -0 3.141592" />
+        <parent link="link_drone_body" />
+        <child link="link_back_camera" />
     </joint>
     <joint name="joint_down_camera" type="fixed">
@@ -426,8 +642,8 @@
         <child link="link_down_camera" />
     </joint>
-    <joint name="joint_down_laser" type="fixed">
-        <origin xyz="-0.01 0.0 0.005" rpy="-0 1.5708 -0" />
-        <parent link="link_drone_body" />
-        <child link="link_down_laser" />
+    <joint name="joint_down_depth" type="fixed">
+        <origin xyz="-0.00 0.0 0.005" rpy="-0 1.5708 -0" />
+        <parent link="link_drone_body" />
+        <child link="link_down_depth" />
     </joint>
     <!-- DRONE STAND JOINTS -->
@@ -475,8 +691,45 @@
     </gazebo>
     <!-- plugin in case we want to control with camera -->
-    <gazebo reference="link_camera">
-        <sensor type="camera" name="camera1">
+    <gazebo reference="link_front_camera">
+        <sensor type="camera" name="camera_front">
             <update_rate>30.0</update_rate>
-            <camera name="front_cam">
+            <camera name="camera_front">
+                <horizontal_fov>1.3962634</horizontal_fov>
+                <image>
+                    <width>800</width>
+                    <height>800</height>
+                    <format>R8G8B8</format>
+                </image>
+                <clip>
+                    <near>0.001</near>
+                    <far>300</far>
+                </clip>
+                <noise>
+                    <type>gaussian</type>
+                    <mean>0.0</mean>
+                    <stddev>0.007</stddev>
+                </noise>
+            </camera>
+            <plugin name="camera_front" filename="libgazebo_ros_camera.so">
+                <alwaysOn>true</alwaysOn>
+                <updateRate>0.0</updateRate>
+                <cameraName>camera_front</cameraName>
+                <imageTopicName>image_raw</imageTopicName>
+                <cameraInfoTopicName>camera_info</cameraInfoTopicName>
+                <frameName>link_front_camera</frameName>
+                <hackBaseline>0.07</hackBaseline>
+                <distortionK1>0.0</distortionK1>
+                <distortionK2>0.0</distortionK2>
+                <distortionK3>0.0</distortionK3>
+                <distortionT1>0.0</distortionT1>
+                <distortionT2>0.0</distortionT2>
+            </plugin>
+        </sensor>
+    </gazebo>
+    <!-- plugin in case we want to control with camera -->
+    <gazebo reference="link_left_camera">
+        <sensor type="camera" name="camera_left">
+            <update_rate>30.0</update_rate>
+            <camera name="camera_left">
                 <horizontal_fov>1.3962634</horizontal_fov>
                 <image>
@@ -495,11 +748,11 @@
                 </noise>
             </camera>
-            <plugin name="front_cam" filename="libgazebo_ros_camera.so">
+            <plugin name="camera_left" filename="libgazebo_ros_camera.so">
                 <alwaysOn>true</alwaysOn>
                 <updateRate>0.0</updateRate>
-                <cameraName>camera1</cameraName>
+                <cameraName>camera_left</cameraName>
                 <imageTopicName>image_raw</imageTopicName>
                 <cameraInfoTopicName>camera_info</cameraInfoTopicName>
-                <frameName>link_camera</frameName>
+                <frameName>link_left_camera</frameName>
                 <hackBaseline>0.07</hackBaseline>
                 <distortionK1>0.0</distortionK1>
@@ -511,8 +764,9 @@
         </sensor>
     </gazebo>
-    <gazebo reference="link_down_camera">
-        <sensor type="camera" name="camera2">
+    <!-- plugin in case we want to control with camera -->
+    <gazebo reference="link_right_camera">
+        <sensor type="camera" name="camera_right">
             <update_rate>30.0</update_rate>
-            <camera name="down_cam">
+            <camera name="camera_right">
                 <horizontal_fov>1.3962634</horizontal_fov>
                 <image>
@@ -531,8 +785,81 @@
                 </noise>
             </camera>
-            <plugin name="down_cam" filename="libgazebo_ros_camera.so">
+            <plugin name="camera_right" filename="libgazebo_ros_camera.so">
                 <alwaysOn>true</alwaysOn>
                 <updateRate>0.0</updateRate>
-                <cameraName>camera2</cameraName>
+                <cameraName>camera_right</cameraName>
+                <imageTopicName>image_raw</imageTopicName>
+                <cameraInfoTopicName>camera_info</cameraInfoTopicName>
+                <frameName>link_right_camera</frameName>
+                <hackBaseline>0.07</hackBaseline>
+                <distortionK1>0.0</distortionK1>
+                <distortionK2>0.0</distortionK2>
+                <distortionK3>0.0</distortionK3>
+                <distortionT1>0.0</distortionT1>
+                <distortionT2>0.0</distortionT2>
+            </plugin>
+        </sensor>
+    </gazebo>
+    <!-- plugin in case we want to control with camera -->
+    <gazebo reference="link_back_camera">
+        <sensor type="camera" name="camera_back">
+        <update_rate>30.0</update_rate>
+            <camera name="camera_back">
+                <horizontal_fov>1.3962634</horizontal_fov>
+                <image>
+                    <width>800</width>
+                    <height>800</height>
+                    <format>R8G8B8</format>
+                </image>
+                <clip>
+                    <near>0.02</near>
+                    <far>300</far>
+                </clip>
+            <noise>
+            <type>gaussian</type>
+            <mean>0.0</mean>
+                    <stddev>0.007</stddev>
+            </noise>
+            </camera>
+            <plugin name="camera_back" filename="libgazebo_ros_camera.so">
+                <alwaysOn>true</alwaysOn>
+                <updateRate>0.0</updateRate>
+                <cameraName>camera_back</cameraName>
+                <imageTopicName>image_raw</imageTopicName>
+                <cameraInfoTopicName>camera_info</cameraInfoTopicName>
+                <frameName>link_back_camera</frameName>
+                <hackBaseline>0.07</hackBaseline>
+                <distortionK1>0.0</distortionK1>
+                <distortionK2>0.0</distortionK2>
+                <distortionK3>0.0</distortionK3>
+                <distortionT1>0.0</distortionT1>
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